File: CS4390.kicad_pcb (KiCad board)
At the start: 2 copper layers, 53 parts, among them J1 Power In, J2 Audio Out, J3 Data In, U1 CS4390, U2 OPA2604, U3 DRV134, U4 DRV134

Commit message: ground plane
Routing:
- net (no net): track 0.00 -> 60.6 mm
- net Net-(C18-Pad2): track 18.2 -> 61.8 mm, vias 0 -> 1
- net Net-(C21-Pad2): track 12.0 -> 49.3 mm
- net +12V: track 148.0 -> 162.2 mm, vias 0 -> 1
- net +5V: track 32.4 -> 40.3 mm
- net GNDA: track 256.0 -> 262.1 mm
- net Net-(R1-Pad1): track 46.7 -> 52.5 mm
- net Net-(C19-Pad2): track 37.8 -> 37.2 mm
- added copper zone on B.Cu, net GNDA
Other:
- board outline added: 97.3 x 51.6 mm

Commit message: V3
Other:
- outline, holes or cut-outs redrawn
Changed lines of the file:
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@@
   (general
     (links 111)
-    (no_connects 7)
+    (no_connects 2)
     (area 104.572999 71.552999 202.005001 123.265001)
     (thickness 1.6)
-    (drawings 29)
+    (drawings 23)
     (tracks 364)
     (zones 0)
@@
   )
   (gr_circle (center 198.882 119.888) (end 200.406 119.888) (layer Edge.Cuts) (width 0.15))
-  (gr_circle (center 140.97 119.888) (end 142.748 119.888) (layer Edge.Cuts) (width 0.15))
   (gr_circle (center 107.95 119.888) (end 109.474 119.888) (layer Edge.Cuts) (width 0.15))
   (gr_circle (center 107.95 74.93) (end 109.474 74.676) (layer Edge.Cuts) (width 0.15))
-  (gr_circle (center 140.97 74.93) (end 142.494 74.93) (layer Edge.Cuts) (width 0.15))
   (gr_circle (center 198.882 74.93) (end 200.152 73.914) (layer Edge.Cuts) (width 0.15))
   (target plus (at 198.95 74.93) (size 5) (width 0.15) (layer Edge.Cuts))
@@
   )
   (gr_circle (center 198.882 119.888) (end 200.152 119.126) (layer F.SilkS) (width 0.2))
-  (gr_circle (center 140.97 120.015) (end 142.24 119.38) (layer F.SilkS) (width 0.2))
   (gr_circle (center 107.95 120.015) (end 109.22 119.38) (layer F.SilkS) (width 0.2))
   (gr_circle (center 107.95 74.93) (end 109.22 75.565) (layer F.SilkS) (width 0.2))
-  (gr_circle (center 140.97 74.93) (end 142.24 75.565) (layer F.SilkS) (width 0.2))
   (gr_line (start 201.93 71.755) (end 201.93 72.39) (angle 90) (layer F.SilkS) (width 0.2))
   (gr_line (start 104.775 71.755) (end 201.93 71.755) (angle 90) (layer F.SilkS) (width 0.2))
@@
   (gr_line (start 201.93 72.39) (end 201.93 122.555) (angle 90) (layer F.SilkS) (width 0.2))
   (target plus (at 198.95 119.93) (size 5) (width 0.15) (layer Edge.Cuts))
-  (target plus (at 140.95 119.93) (size 5) (width 0.15) (layer Edge.Cuts))
   (target plus (at 107.95 74.93) (size 5) (width 0.15) (layer Edge.Cuts))
-  (target plus (at 140.95 74.93) (size 5) (width 0.15) (layer Edge.Cuts))
   (target plus (at 107.95 119.93) (size 5) (width 0.15) (layer Edge.Cuts))
   (segment (start 121.666 91.064) (end 121.666 117.094) (width 0.7) (layer B.Cu) (net 0))
@@
     (polygon
       (pts
-        (xy 144.272 77.978) (xy 137.668 77.978) (xy 137.668 71.628) (xy 144.272 71.628)
-      )
-    )
-  )
-  (zone (net 0) (net_name "") (layer F.Cu) (hatch edge 0.508)
-    (connect_pads (clearance 0.508))
-    (min_thickness 0.254)
-    (keepout (tracks not_allowed) (vias not_allowed) (copperpour allowed))
-    (fill (arc_segments 16) (thermal_gap 0.508) (thermal_bridge_width 0.508))
-    (polygon
-      (pts
         (xy 110.998 77.978) (xy 104.902 77.978) (xy 104.648 77.724) (xy 104.648 71.628) (xy 110.998 71.628)
       )
@@
     (polygon
       (pts
-        (xy 144.018 123.19) (xy 137.922 123.19) (xy 137.922 116.84) (xy 144.018 116.84)
-      )
-    )
-  )
-  (zone (net 0) (net_name "") (layer F.Cu) (hatch edge 0.508)
-    (connect_pads (clearance 0.508))
-    (min_thickness 0.254)
-    (keepout (tracks not_allowed) (vias not_allowed) (copperpour allowed))
-    (fill (arc_segments 16) (thermal_gap 0.508) (thermal_bridge_width 0.508))
-    (polygon
-      (pts
         (xy 201.93 123.19) (xy 195.834 123.19) (xy 195.834 116.84) (xy 201.93 116.84)
-      )
-    )
-  )
-  (zone (net 4) (net_name GNDA) (layer B.Cu) (hatch edge 0.508)
-    (connect_pads (clearance 0.508))
-    (min_thickness 0.254)
-    (fill yes (arc_segments 16) (thermal_gap 0.508) (thermal_bridge_width 0.508))
-    (polygon
-      (pts
-        (xy 128.778 77.978) (xy 128.778 84.582) (xy 139.192 84.582) (xy 140.208 85.344) (xy 145.034 80.518)
-        (xy 156.718 80.518) (xy 156.718 74.93) (xy 128.778 74.93) (xy 128.778 78.486)
       )
     )
@@
       )
     )
-  )
-  (zone (net 4) (net_name GNDA) (layer B.Cu) (hatch edge 0.508)
-    (connect_pads (clearance 0.508))
-    (min_thickness 0.254)
-    (fill yes (arc_segments 16) (thermal_gap 0.508) (thermal_bridge_width 0.508))
-    (polygon
-      (pts
-        (xy 148.59 122.174) (xy 148.59 118.618) (xy 143.764 113.792) (xy 140.208 113.792) (xy 139.192 114.808)
-        (xy 128.27 114.808) (xy 128.27 122.174)
-      )
-    )

Commit message: pre-trace
Parts:
- added J4: Power In, Pin_Headers:Pin_Header_Straight_1x04_Pitch2.54mm, F.Cu at (153.4, 133.3)
- added J5: Left, Connectors_Terminal_Blocks:TerminalBlock_Altech_AK300-3_P5.00mm, F.Cu at (153.4, 133.3)
- added J6: Right, Connectors_Terminal_Blocks:TerminalBlock_Altech_AK300-3_P5.00mm, F.Cu at (153.4, 133.3)
- C11: value 0.1uF -> 220pF
- C2: value 10uF -> 0.1uF
- C3: value 1nF -> 10uF
- C7: value 220pF -> 1nF
- D1, D2, D3, D4: footprint Diodes_THT:D_A-405_P10.16mm_Horizontal -> Diodes_THT:D_DO-35_SOD27_P2.54mm_Vertical_AnodeUp
- J1: value Power In -> GS3; footprint Pin_Headers:Pin_Header_Straight_1x05_Pitch2.54mm -> Connectors:GS3
- J2: value Audio Out -> GS3; footprint Pin_Headers:Pin_Header_Straight_1x05_Pitch2.54mm -> Connectors:GS3
- R1, R10, R11, R12, R13, R2, R3, R4, R5, R6, R7, R8, R9: footprint Resistors_THT:R_Axial_DIN0207_L6.3mm_D2.5mm_P10.16mm_Horizontal -> Resistors_THT:R_Axial_DIN0204_L3.6mm_D1.6mm_P2.54mm_Vertical
- U1: value CS4390 -> OPA2604; footprint Housings_DIP:DIP-20_W7.62mm_LongPads -> Housings_DIP:DIP-8_W7.62mm_LongPads
- U2: value OPA2604 -> CS4390; footprint Housings_DIP:DIP-8_W7.62mm_LongPads -> Housings_DIP:DIP-20_W7.62mm_LongPads
- moved R15 66.9 mm to (153.4, 133.3), turned to 0 degrees
- moved FL4 64.8 mm to (153.4, 133.3), turned to 0 degrees
- moved J1 60.3 mm to (153.4, 133.3), turned to 0 degrees
- moved C14 59.2 mm to (153.4, 133.3), turned to 0 degrees
- moved D1 58.9 mm to (153.4, 133.3), turned to 0 degrees
- moved C1 58.5 mm to (153.4, 133.3), turned to 0 degrees
- moved U1 58.4 mm to (153.4, 133.3)
- moved R14 58.1 mm to (153.4, 133.3)
- moved FL3 57.9 mm to (153.4, 133.3), turned to 0 degrees
- moved J2 57.2 mm to (153.4, 133.3)
- moved C15 57.1 mm to (153.4, 133.3), turned to 0 degrees
- moved D3 56.7 mm to (153.4, 133.3), turned to 0 degrees
- moved R1 56.4 mm to (153.4, 133.3), turned to 0 degrees
- moved FL2 55.2 mm to (153.4, 133.3), turned to 0 degrees
- moved C2 52.8 mm to (153.4, 133.3), turned to 0 degrees
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Connections:
- C1 pad 1: +5V -> +15V
- C1 pad 2: GND -> -12V
- C10 pad 2: GNDA -> Net-(C10-Pad2)
- C11 pad 1: +12V -> Net-(C11-Pad1)
- C13 pad 1: Net-(C13-Pad1) -> Net-(C10-Pad1)
- C14 pad 2: +12V -> +15V
- C16 pad 2: +12V -> +15V
- C2 pad 2: GND -> GNDA
- C3 pad 1: Net-(C3-Pad1) -> +5V
- C7 pad 1: Net-(C13-Pad1) -> Net-(C7-Pad1)
- C7 pad 2: Net-(C7-Pad2) -> GNDA
- C8 pad 1: Net-(C8-Pad1) -> Net-(C12-Pad1)
- C8 pad 2: GNDA -> Net-(C8-Pad2)
- C9 pad 1: Net-(C12-Pad1) -> Net-(C9-Pad1)
- C9 pad 2: Net-(C9-Pad2) -> GNDA
- D1 pad 1: +12V -> +15V
- D2 pad 1: +12V -> +15V
- D3 pad 1: +12V -> +15V
- D4 pad 1: +12V -> +15V
- FL1 pad 1: Net-(C20-Pad2) -> Net-(C18-Pad2)
- FL1 pad 3: R+ -> Net-(FL1-Pad3)
- FL2 pad 1: Net-(C21-Pad2) -> Net-(C19-Pad2)
- FL2 pad 3: R- -> Net-(FL2-Pad3)
- FL3 pad 1: Net-(C18-Pad2) -> Net-(C20-Pad2)
- FL3 pad 3: L+ -> Net-(FL3-Pad3)
- FL4 pad 1: Net-(C19-Pad2) -> Net-(C21-Pad2)
- FL4 pad 3: L- -> Net-(FL4-Pad3)
- J1 pad 1: GNDA -> Net-(J1-Pad1)
- J1 pad 2: -12V -> Net-(J1-Pad2)
- J1 pad 3: +12V -> GNDA
- J2 pad 1: L+ -> Net-(J1-Pad1)
- J2 pad 2: L- -> Net-(J2-Pad2)
- J2 pad 3: (no net) -> GNDA
- R1 pad 1: Net-(R1-Pad1) -> Net-(J1-Pad1)
- R10 pad 1: Net-(C5-Pad1) -> Net-(C6-Pad1)
- R10 pad 2: Net-(C7-Pad2) -> Net-(C8-Pad2)
- R11 pad 1: Net-(C3-Pad1) -> Net-(C4-Pad1)
- R11 pad 2: Net-(C8-Pad1) -> Net-(C9-Pad1)
- R12 pad 1: Net-(C6-Pad1) -> Net-(C7-Pad1)
- R12 pad 2: Net-(C9-Pad2) -> Net-(C10-Pad2)
- R13 pad 1: Net-(C4-Pad1) -> Net-(C5-Pad1)
- R13 pad 2: Net-(C10-Pad1) -> Net-(C11-Pad1)
- R2 pad 1: Net-(C3-Pad1) -> Net-(C6-Pad1)
- R3 pad 1: Net-(C5-Pad1) -> Net-(C4-Pad1)
- R4 pad 1: Net-(C4-Pad1) -> Net-(C7-Pad1)
- R5 pad 1: Net-(C6-Pad1) -> Net-(C5-Pad1)
- R6 pad 1: Net-(C13-Pad1) -> Net-(C12-Pad1)
- R6 pad 2: Net-(C5-Pad1) -> Net-(C6-Pad1)
- R7 pad 1: Net-(C3-Pad1) -> Net-(C4-Pad1)
- R8 pad 1: Net-(C12-Pad1) -> Net-(C10-Pad1)
- R8 pad 2: Net-(C6-Pad1) -> Net-(C7-Pad1)
- R9 pad 1: Net-(C4-Pad1) -> Net-(C5-Pad1)
- U1 pad 1: GNDA -> Net-(C10-Pad1)
- U1 pad 2: Net-(R1-Pad1) -> Net-(C10-Pad2)
- U1 pad 3: +5V -> Net-(C11-Pad1)
- U1 pad 4: GNDA -> -12V
- U1 pad 5: GND -> Net-(C9-Pad1)
- U1 pad 6: +5V -> Net-(C8-Pad2)
- U1 pad 7: LRCK -> Net-(C12-Pad1)
- U1 pad 8: MCLK -> +15V
- U2 pad 1: Net-(C13-Pad1) -> GNDA
- U2 pad 2: Net-(C8-Pad1) -> Net-(J1-Pad1)
- U2 pad 3: Net-(C7-Pad2) -> +5V
- U2 pad 5: Net-(C9-Pad2) -> GNDA
- U2 pad 6: Net-(C10-Pad1) -> +5V
- U2 pad 7: Net-(C12-Pad1) -> LRCK
- U2 pad 8: +12V -> MCLK
- U3 pad 4: Net-(C13-Pad2) -> Net-(C12-Pad2)
- U3 pad 6: +12V -> +15V
- U4 pad 3: (no net) -> GNDA
- U4 pad 4: Net-(C12-Pad2) -> Net-(C13-Pad2)
- U4 pad 6: +12V -> +15V
Routing:
- net GNDA: track 262.1 -> 0.00 mm
- net +12V: track 162.2 -> 0.00 mm, vias 1 -> 0
- net -12V: track 99.3 -> 0.00 mm
- net Net-(C18-Pad2): track 61.8 -> 0.00 mm, vias 1 -> 0
- net (no net): track 60.6 -> 0.00 mm
- net Net-(R1-Pad1): track 52.5 -> 0.00 mm
- net Net-(C21-Pad2): track 49.3 -> 0.00 mm
- net +5V: track 40.3 -> 0.00 mm
- net Net-(C19-Pad2): track 37.2 -> 0.00 mm
- net GND: track 35.1 -> 0.00 mm
- net Net-(C8-Pad1): track 32.4 -> 0.00 mm
- net Net-(C10-Pad1): track 31.6 -> 0.00 mm
- net Net-(C3-Pad1): track 31.3 -> 0.00 mm
- net Net-(C6-Pad1): track 29.1 -> 0.00 mm
- net Net-(C12-Pad1): track 24.0 -> 0.00 mm
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- removed copper zone on B.Cu, net GNDA
Other:
- board size 97.3 x 51.6 mm -> 97.2 x 51.4 mm
- board text removed: "Zose analog output board"

Commit message: base placement
Parts:
- J5, J6: footprint Connectors_Terminal_Blocks:TerminalBlock_Altech_AK300-3_P5.00mm -> Connectors_Molex:Molex_SPOX-5267_22-03-5035_03x2.54mm_Straight
- moved R15 68.5 mm to (199.4, 82.5), turned to 180 degrees
- moved C2 63.6 mm to (116.8, 81.2), turned to 90 degrees
- moved C19 62.8 mm to (176.6, 74.9)
- moved R14 62.0 mm to (182.9, 78.7)
- moved C1 60.7 mm to (110.5, 90.2), turned to 270 degrees
- moved C3 60.1 mm to (123.2, 81.3), turned to 90 degrees
- moved D1 58.9 mm to (185.4, 83.8), turned to 180 degrees
- moved J4 58.3 mm to (115.6, 88.9)
- moved U2 57.9 mm to (119.4, 86.4)
- moved C14 57.6 mm to (161.4, 76.2)
- moved C17 57.1 mm to (156.2, 76.2), turned to 180 degrees
- moved U3 56.9 mm to (176.5, 81.3), turned to 270 degrees
- moved J5 56.7 mm to (193.0, 92.7), turned to 90 degrees
- moved FL2 54.4 mm to (182.9, 87.6)
- moved C4 51.5 mm to (132.1, 86.4), turned to 90 degrees
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Routing:
- net GNDA: track 0.00 -> 74.8 mm
- net Net-(C20-Pad2): track 0.00 -> 27.0 mm
- net Net-(C18-Pad2): track 0.00 -> 23.0 mm
- net Net-(C21-Pad2): track 0.00 -> 23.0 mm
- net Net-(C19-Pad2): track 0.00 -> 22.4 mm
- net Net-(C9-Pad1): track 0.00 -> 18.3 mm
- net Net-(C12-Pad1): track 0.00 -> 17.6 mm
- net Net-(C4-Pad1): track 0.00 -> 16.8 mm
- net Net-(C10-Pad1): track 0.00 -> 16.7 mm
- net Net-(C8-Pad2): track 0.00 -> 16.4 mm
- net Net-(C11-Pad1): track 0.00 -> 16.4 mm
- net Net-(C7-Pad1): track 0.00 -> 14.1 mm
- net Net-(C6-Pad1): track 0.00 -> 11.2 mm
- net Net-(C5-Pad1): track 0.00 -> 11.2 mm
- net Net-(C21-Pad1): track 0.00 -> 9.45 mm
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
Commit message: gerber
Parts:
- removed J1, J2: GS3, Connectors:GS3
- moved C1 37.3 mm to (147.8, 89.6), turned to 90 degrees
- moved C17 36.8 mm to (156.2, 113.0), turned to 270 degrees
- moved C15 19.1 mm to (158.8, 94.0)
- moved C16 16.7 mm to (163.8, 102.9), turned to 180 degrees
- moved C9 16.6 mm to (143.4, 85.1)
- moved C8 16.2 mm to (138.5, 95.2), turned to 0 degrees
- moved C10 14.4 mm to (138.5, 110.5), turned to 0 degrees
- moved C13 13.0 mm to (152.4, 109.2), turned to 0 degrees
- moved C12 11.4 mm to (152.5, 87.6), turned to 0 degrees
- moved C19 10.5 mm to (166.4, 77.5)
- moved C11 9.98 mm to (143.5, 100.3), turned to 180 degrees
- moved C5 9.75 mm to (135.9, 100.3), turned to 180 degrees
- moved C6 9.67 mm to (135.9, 95.2), turned to 180 degrees
- moved C20 7.70 mm to (166.4, 119.4)
- moved C18 7.62 mm to (167.7, 95.2)
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Routing:
- net +15V: track 0.00 -> 207.1 mm, vias 0 -> 2
- net -12V: track 0.00 -> 103.0 mm, vias 0 -> 2
- net +5V: track 3.81 -> 53.2 mm
- net Net-(C10-Pad2): track 0.00 -> 28.8 mm
- net Net-(J1-Pad1): track 0.00 -> 25.1 mm
- net Net-(C10-Pad1): track 16.7 -> 29.2 mm, vias 0 -> 1
- net Net-(C12-Pad1): track 17.6 -> 25.4 mm
- net Net-(C6-Pad1): track 11.2 -> 6.35 mm
- net Net-(C4-Pad1): track 16.8 -> 12.7 mm
- net Net-(C7-Pad1): track 14.1 -> 16.8 mm
- net GNDA: track 74.8 -> 72.1 mm
- net SDATA: track 3.81 -> 6.35 mm
- net MCLK: track 3.81 -> 6.35 mm
- net LRCK: track 3.81 -> 6.35 mm
- net BCLK: track 3.81 -> 6.35 mm
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- added copper zone on B.Cu, net GNDA
- added copper zone on F.Cu, net GNDA
Other:
- net class Default: clearance 0.2 -> 0.5
- rule trace_clearance: 0.2 -> 0.5

Commit message: retrace
Parts:
- removed C14: 1uF, Capacitors_THT:C_Rect_L7.2mm_W3.5mm_P5.00mm_FKS2_FKP2_MKS2_MKP2
- moved R14 19.1 mm to (183.4, 96.0)
- moved C2 18.0 mm to (114.3, 99.1)
- moved R17 16.2 mm to (193.5, 104.1)
- moved C3 12.8 mm to (114.3, 90.4)
- moved J4 11.2 mm to (121.4, 80.3), turned to 270 degrees
- moved C19 9.95 mm to (173.2, 84.8), turned to 90 degrees
- moved C20 8.80 mm to (173.2, 113.9), turned to 270 degrees
- moved C1 8.53 mm to (152.7, 82.5), turned to 180 degrees
- moved J6 5.79 mm to (189.0, 113.8)
- moved D4 5.55 mm to (179.3, 118.4)
- moved C15 5.35 mm to (164.1, 95.0), turned to 180 degrees
- moved FL3 4.82 mm to (176.8, 113.8)
- moved FL4 4.82 mm to (176.8, 108.7)
- moved R16 4.44 mm to (183.4, 118.4)
- moved D2 4.10 mm to (179.3, 104.1)
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Routing:
- net GNDA: track 72.1 -> 17.7 mm
- net +15V: track 207.1 -> 172.3 mm, vias 2 -> 0
- net -12V: track 103.0 -> 116.2 mm, vias 2 -> 0
- net Net-(C20-Pad2): track 27.1 -> 17.0 mm
- net Net-(J1-Pad1): track 25.1 -> 34.3 mm
- net Net-(C6-Pad1): track 6.35 -> 12.7 mm
- net Net-(C18-Pad2): track 23.0 -> 17.7 mm
- net Net-(C21-Pad2): track 23.0 -> 18.2 mm
- net Net-(C19-Pad2): track 22.7 -> 18.3 mm
- net Net-(FL4-Pad3): track 5.08 -> 7.11 mm
- net Net-(FL3-Pad3): track 5.08 -> 7.11 mm
- net Net-(FL2-Pad3): track 5.08 -> 7.11 mm
- net Net-(FL1-Pad3): track 5.08 -> 7.11 mm
- net Net-(C19-Pad1): track 6.50 -> 8.52 mm
- net +5V: track 53.2 -> 51.5 mm
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Other:
- outline, holes or cut-outs redrawn
- board text added: "+"
- board text added: "-"
- board text added: "5V"
- board text added: "BCLK"
- board text added: "DATA"
- board text added: "G"
- board text added: "LRCK"
- board text added: "MCLK"
- board text added: "Rev. A (201804)"
- board text added: "ZOSE Line out board"
