File: CS4390.kicad_pcb (KiCad board)
At the start: 2 copper layers, 97.2 x 51.4 mm, 53 parts, among them J3 Data In, J4 Power In, J5 Left, J6 Right, U1 OPA2604, U2 CS4390, U3 DRV134, U4 DRV134

Commit message: ready for prod
Parts:
- removed C17: 1uF, Capacitors_THT:C_Rect_L7.2mm_W3.5mm_P5.00mm_FKS2_FKP2_MKS2_MKP2
- added J1: GS3, Wire_Pads:SolderWirePad_3x_0-8mmDrill, F.Cu at (127.0, 75.7)
- added J2: GS3, Wire_Pads:SolderWirePad_3x_0-8mmDrill, F.Cu at (131.7, 78.1)
Routing:
- net Net-(J1-Pad1): track 34.3 -> 66.6 mm
- net GNDA: track 17.7 -> 32.7 mm
- net Net-(J2-Pad2): track 0.00 -> 13.0 mm
- net Net-(J1-Pad2): track 0.40 -> 12.4 mm
- net -12V: track 116.2 -> 111.3 mm
Other:
- board text added: "IGN Rev. A"
- board text removed: "Rev. A (201804)"
Changed lines of the file:
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@@
 (kicad_pcb (version 4) (host pcbnew 4.0.7)
   (general
-    (links 113)
-    (no_connects 1)
+    (links 117)
+    (no_connects 0)
     (area 104.699999 71.679999 202.005001 123.265001)
     (thickness 1.6)
     (drawings 22)
-    (tracks 248)
+    (tracks 269)
     (zones 0)
-    (modules 53)
+    (modules 54)
     (nets 40)
   )
@@
     (visible_elements 7FFFEFFF)
     (pcbplotparams
-      (layerselection 0x290a0_80000001)
+      (layerselection 0x010a0_80000001)
       (usegerberextensions false)
       (excludeedgelayer true)
@@
     (add_net SDATA)
   )
+  (module Wire_Pads:SolderWirePad_3x_0-8mmDrill (layer F.Cu)
+    (at 131.699 78.105 180)
+    (fp_text reference J2 (at -5.588 0 180) (layer F.SilkS)
+      (effects (font (size 1 1) (thickness 0.15)))
+    )
+    (fp_text value GS3 (at 0 2.54 180) (layer F.Fab)
+      (effects (font (size 1 1) (thickness 0.15)))
+    )
+    (pad 1 thru_hole circle (at -3.175 0 180) (size 1.99898 1.99898) (drill 0.8001) (layers *.Cu *.Mask)
+      (net 37 "Net-(J1-Pad1)"))
+    (pad 2 thru_hole circle (at 0 0 180) (size 1.99898 1.99898) (drill 0.8001) (layers *.Cu *.Mask)
+      (net 39 "Net-(J2-Pad2)"))
+    (pad 3 thru_hole circle (at 3.175 0 180) (size 1.99898 1.99898) (drill 0.8001) (layers *.Cu *.Mask)
+      (net 2 GNDA))
+  )
+  (module Wire_Pads:SolderWirePad_3x_0-8mmDrill (layer F.Cu)
+    (at 127 75.692 180)
+    (fp_text reference J1 (at -5.715 -0.127 180) (layer F.SilkS)
+      (effects (font (size 1 1) (thickness 0.15)))
+    )
+    (fp_text value GS3 (at 0 2.54 180) (layer F.Fab)
+      (effects (font (size 1 1) (thickness 0.15)))
+    )
+    (pad 1 thru_hole circle (at -3.175 0 180) (size 1.99898 1.99898) (drill 0.8001) (layers *.Cu *.Mask)
+      (net 37 "Net-(J1-Pad1)"))
+    (pad 2 thru_hole circle (at 0 0 180) (size 1.99898 1.99898) (drill 0.8001) (layers *.Cu *.Mask)
+      (net 38 "Net-(J1-Pad2)"))
+    (pad 3 thru_hole circle (at 3.175 0 180) (size 1.99898 1.99898) (drill 0.8001) (layers *.Cu *.Mask)
+      (net 2 GNDA))
+  )
   (module Diodes_THT:D_DO-35_SOD27_P2.54mm_Vertical_AnodeUp (layer F.Cu)
     (at 179.324 118.364 180)
@@
     (pad 2 thru_hole circle (at 5 0 180) (size 1.6 1.6) (drill 0.8) (layers *.Cu *.Mask)
       (net 27 +15V))
-    (model ${KISYS3DMOD}/Capacitors_THT.3dshapes/C_Rect_L7.2mm_W3.5mm_P5.00mm_FKS2_FKP2_MKS2_MKP2.wrl
-      (at (xyz 0 0 0))
-      (scale (xyz 1 1 1))
-      (rotate (xyz 0 0 0))
-    )
-  )
-  (module Capacitors_THT:C_Rect_L7.2mm_W3.5mm_P5.00mm_FKS2_FKP2_MKS2_MKP2 (layer F.Cu)
-    (at 157.48 113.919 180)
-    (descr "C, Rect series, Radial, pin pitch=5.00mm, , length*width=7.2*3.5mm^2, Capacitor, http://www.wima.com/EN/WIMA_FKS_2.pdf")
-    (tags "C Rect series Radial pin pitch 5.00mm  length 7.2mm width 3.5mm Capacitor")
-    (fp_text reference C17 (at 2.4257 -0.0254 180) (layer F.SilkS)
-      (effects (font (size 1 1) (thickness 0.15)))
-    )
-    (fp_text value 1uF (at 2.5 3.06 180) (layer F.Fab)
-      (effects (font (size 1 1) (thickness 0.15)))
-    )
-    (fp_line (start -1.1 -1.75) (end -1.1 1.75) (layer F.Fab) (width 0.1))
-    (fp_line (start -1.1 1.75) (end 6.1 1.75) (layer F.Fab) (width 0.1))
-    (fp_line (start 6.1 1.75) (end 6.1 -1.75) (layer F.Fab) (width 0.1))
-    (fp_line (start 6.1 -1.75) (end -1.1 -1.75) (layer F.Fab) (width 0.1))
-    (fp_line (start -1.16 -1.81) (end 6.16 -1.81) (layer F.SilkS) (width 0.12))
-    (fp_line (start -1.16 1.81) (end 6.16 1.81) (layer F.SilkS) (width 0.12))
-    (fp_line (start -1.16 -1.81) (end -1.16 1.81) (layer F.SilkS) (width 0.12))
-    (fp_line (start 6.16 -1.81) (end 6.16 1.81) (layer F.SilkS) (width 0.12))
-    (fp_line (start -1.45 -2.1) (end -1.45 2.1) (layer F.CrtYd) (width 0.05))
-    (fp_line (start -1.45 2.1) (end 6.45 2.1) (layer F.CrtYd) (width 0.05))
-    (fp_line (start 6.45 2.1) (end 6.45 -2.1) (layer F.CrtYd) (width 0.05))
-    (fp_line (start 6.45 -2.1) (end -1.45 -2.1) (layer F.CrtYd) (width 0.05))
-    (fp_text user %R (at 2.54 0 180) (layer F.Fab)
-      (effects (font (size 1 1) (thickness 0.15)))
-    )
-    (pad 1 thru_hole circle (at 0 0 180) (size 1.6 1.6) (drill 0.8) (layers *.Cu *.Mask)
-      (net 2 GNDA))
-    (pad 2 thru_hole circle (at 5 0 180) (size 1.6 1.6) (drill 0.8) (layers *.Cu *.Mask)
-      (net 10 -12V))
     (model ${KISYS3DMOD}/Capacitors_THT.3dshapes/C_Rect_L7.2mm_W3.5mm_P5.00mm_FKS2_FKP2_MKS2_MKP2.wrl
       (at (xyz 0 0 0))
@@
     (effects (font (size 1.5 1.5) (thickness 0.3)))
   )
-  (gr_text "Rev. A (201804)" (at 122.428 119.888) (layer F.SilkS)
+  (gr_text "IGN Rev. A " (at 122.428 119.888) (layer F.SilkS)
     (effects (font (size 1.5 1.5) (thickness 0.3)))
   )
@@
   (segment (start 119.78 91.44) (end 119.38 91.44) (width 0.7) (layer F.Cu) (net 1) (status 30))
   (segment (start 114.22 90.344) (end 114.3 90.424) (width 0.7) (layer F.Cu) (net 1) (status 30))
+  (segment (start 123.825 75.692) (end 120.904 75.692) (width 0.7) (layer F.Cu) (net 2))
+  (segment (start 120.904 75.692) (end 116.332 80.264) (width 0.7) (layer F.Cu) (net 2))
+  (segment (start 123.825 75.692) (end 126.238 78.105) (width 0.7) (layer F.Cu) (net 2))
+  (segment (start 126.238 78.105) (end 128.524 78.105) (width 0.7) (layer F.Cu) (net 2))
   (segment (start 116.332 80.264) (end 116.332 81.28) (width 0.7) (layer B.Cu) (net 2))
   (segment (start 114.3 83.312) (end 114.3 85.424) (width 0.7) (layer B.Cu) (net 2))
@@
   (segment (start 157.4 109.22) (end 160.02 109.22) (width 0.7) (layer F.Cu) (net 9))
   (segment (start 160.02 109.22) (end 161.29 107.95) (width 0.7) (layer F.Cu) (net 9))
+  (segment (start 154.94 111.459) (end 159.051 115.57) (width 0.7) (layer B.Cu) (net 10))
+  (segment (start 159.051 115.57) (end 161.29 115.57) (width 0.7) (layer B.Cu) (net 10))
   (segment (start 113.792 80.264) (end 113.792 81.026) (width 0.7) (layer F.Cu) (net 10))
   (segment (start 113.792 81.026) (end 115.316 82.55) (width 0.7) (layer F.Cu) (net 10))
@@
   (segment (start 145.66999 84.53401) (end 146.854001 83.349999) (width 0.7) (layer B.Cu) (net 10))
   (segment (start 146.854001 83.349999) (end 147.654 82.55) (width 0.7) (layer B.Cu) (net 10))
-  (segment (start 152.48 113.919) (end 152.781 113.919) (width 0.7) (layer B.Cu) (net 10))
-  (segment (start 152.781 113.919) (end 154.432 115.57) (width 0.7) (layer B.Cu) (net 10))
-  (segment (start 154.432 115.57) (end 161.29 115.57) (width 0.7) (layer B.Cu) (net 10))
   (segment (start 154.94 101.6) (end 154.94 111.459) (width 0.7) (layer B.Cu) (net 10))
-  (segment (start 154.94 111.459) (end 152.48 113.919) (width 0.7) (layer B.Cu) (net 10))
   (segment (start 147.654 82.55) (end 147.654 82.804) (width 0.7) (layer B.Cu) (net 10) (status 30))
   (segment (start 161.29 88.9) (end 161.29 90.678) (width 0.7) (layer B.Cu) (net 10))
@@
   (segment (start 181.864 113.792) (end 188.976 113.792) (width 0.7) (layer F.Cu) (net 35) (status 10))
   (segment (start 181.864 108.712) (end 188.976 108.712) (width 0.7) (layer F.Cu) (net 36) (status 10))
+  (segment (start 130.175 75.692) (end 128.325509 73.842509) (width 0.7) (layer B.Cu) (net 37))
+  (segment (start 122.937243 73.842509) (end 121.975509 74.804243) (width 0.7) (layer B.Cu) (net 37))
+  (segment (start 128.325509 73.842509) (end 122.937243 73.842509) (width 0.7) (layer B.Cu) (net 37))
+  (segment (start 121.975509 74.804243) (end 121.975509 77.597507) (width 0.7) (layer B.Cu) (net 37))
+  (segment (start 121.975509 77.597507) (end 123.112001 78.733999) (width 0.7) (layer B.Cu) (net 37))
+  (segment (start 123.112001 78.733999) (end 123.112001 87.067999) (width 0.7) (layer B.Cu) (net 37))
+  (segment (start 123.112001 87.067999) (end 121.28 88.9) (width 0.7) (layer B.Cu) (net 37))
+  (segment (start 121.28 88.9) (end 119.38 88.9) (width 0.7) (layer B.Cu) (net 37))
+  (segment (start 130.175 75.692) (end 132.461 75.692) (width 0.7) (layer F.Cu) (net 37))
+  (segment (start 132.461 75.692) (end 134.874 78.105) (width 0.7) (layer F.Cu) (net 37))
   (segment (start 127 99.06) (end 125.984 99.06) (width 0.7) (layer B.Cu) (net 37))
   (segment (start 125.984 99.06) (end 124.46 100.584) (width 0.7) (layer B.Cu) (net 37))
@@
   (segment (start 121.28 88.9) (end 124.94999 92.56999) (width 0.7) (layer F.Cu) (net 37))
   (segment (start 124.94999 92.56999) (end 124.94999 94.86999) (width 0.7) (layer F.Cu) (net 37))
+  (segment (start 127 75.692) (end 126.000511 76.691489) (width 0.7) (layer B.Cu) (net 38))
+  (segment (start 126.000511 76.691489) (end 126.000511 83.860511) (width 0.7) (layer B.Cu) (net 38))
+  (segment (start 126.000511 83.860511) (end 127 84.86) (width 0.7) (layer B.Cu) (net 38))
+  (segment (start 127 84.86) (end 127 86.36) (width 0.7) (layer B.Cu) (net 38))
+  (segment (start 127 86.36) (end 127 86.868) (width 0.7) (layer F.Cu) (net 38))
   (segment (start 127 86.36) (end 126.6 86.36) (width 0.7) (layer F.Cu) (net 38) (status 30))
+  (segment (start 131.699 78.105) (end 129.05001 80.75399) (width 0.7) (layer B.Cu) (net 39))
+  (segment (start 129.05001 80.75399) (end 129.05001 87.24999) (width 0.7) (layer B.Cu) (net 39))
+  (segment (start 129.05001 87.24999) (end 127.4 88.9) (width 0.7) (layer B.Cu) (net 39))
+  (segment (start 127.4 88.9) (end 127 88.9) (width 0.7) (layer B.Cu) (net 39))
   (zone (net 0) (net_name "") (layer F.Cu) (hatch edge 0.508)
     (connect_pads (clearance 0.508))
