File: CS4390.kicad_pcb (KiCad board)
At the start: 2 copper layers, 97.2 x 51.4 mm, 54 parts, among them J1 GS3, J2 GS3, J3 Data In, J4 Power In, J5 Left, J6 Right, U1 OPA2604, U2 CS4390, U3 DRV134, U4 DRV134

Commit message: Rev B
Parts:
- moved U1 11.1 mm to (155.2, 93.7), turned to 270 degrees
Connections:
- net -12V renamed -15V
- net Net-(C4-Pad1) renamed L+
- net Net-(C5-Pad1) renamed R+
- net Net-(C6-Pad1) renamed L-
- net Net-(C7-Pad1) renamed R-
- J1 pad 1: Net-(J1-Pad1) -> CTRL
- J2 pad 1: Net-(J1-Pad1) -> CTRL
- R1 pad 1: Net-(J1-Pad1) -> CTRL
- U1 pad 1: Net-(C10-Pad1) -> Net-(C12-Pad1)
- U1 pad 2: Net-(C10-Pad2) -> Net-(C8-Pad2)
- U1 pad 3: Net-(C11-Pad1) -> Net-(C9-Pad1)
- U1 pad 5: Net-(C9-Pad1) -> Net-(C11-Pad1)
- U1 pad 6: Net-(C8-Pad2) -> Net-(C10-Pad2)
- U1 pad 7: Net-(C12-Pad1) -> Net-(C10-Pad1)
- U2 pad 1: GNDA -> CTRL
- U2 pad 11: Net-(J1-Pad1) -> CTRL
- U2 pad 12: Net-(J1-Pad1) -> CTRL
- U2 pad 15: Net-(J1-Pad1) -> CTRL
- U2 pad 16: Net-(J1-Pad1) -> CTRL
- U2 pad 2: Net-(J1-Pad1) -> CTRL
Routing:
- net CTRL: track 0.00 -> 68.6 mm
- net Net-(J1-Pad1): track 66.6 -> 0.00 mm
- net Net-(C10-Pad2): track 28.8 -> 12.9 mm
- net -15V: track 111.3 -> 95.8 mm
- net +15V: track 172.3 -> 162.5 mm
- net Net-(C9-Pad1): track 18.2 -> 13.1 mm
- net Net-(C12-Pad1): track 25.4 -> 30.5 mm
- net Net-(C11-Pad1): track 14.0 -> 9.03 mm
- net R+: track 12.2 -> 16.0 mm
- net GNDA: track 32.7 -> 29.5 mm
- net SDATA: track 5.80 -> 7.16 mm
- net Net-(C8-Pad2): track 14.0 -> 14.9 mm
- net +5V: track 51.5 -> 50.6 mm
- net Net-(C10-Pad1): track 28.4 -> 27.6 mm
- net R-: track 16.8 -> 16.3 mm
Other:
- board text added: "Rev. B"
- board text removed: "IGN Rev. A"
