File: CS4390.sch (KiCad schematic (older format))
At the start: 53 parts, among them J1 Power In, J2 Audio Out, J3 Data In, U1 CS4390, U2 OPA2604, U3 DRV134, U4 DRV134

Commit message: V3
Parts:
- removed J1: Power In, Pin_Headers:Pin_Header_Straight_1x05_Pitch2.54mm, symbol Conn_01x05
- removed J2: Audio Out, Pin_Headers:Pin_Header_Straight_1x05_Pitch2.54mm, symbol Conn_01x05
- added J1, J2: GS3, Connectors:GS3, symbol GS3
- added J4: Power In, symbol Conn_01x04
- added J5: Left, symbol Screw_Terminal_01x03
- added J6: Right, symbol Screw_Terminal_01x03
- renumbered C11 to C1, C9 to C10, C10 to C11, C13 to C12, C12 to C13, C1 to C2, C2 to C3, C3 to C4, C4 to C5, C5 to C6, C6 to C7, C7 to C8, C8 to C9, FL3 to FL1, FL4 to FL2, FL1 to FL3, FL2 to FL4, U2 to U1, U1 to U2
Connections:
- net GND is gone; now on net GNDA: C2.2, C3.2, U2.5 (DGND)
- net +5V: now also J4.2 (Pin_2)
- net -12V: now also C1.2, U1.4 (V-), J4.4 (Pin_4)
- net GNDA: now also U4.3 (-), J1.3 (G3), J2.3 (G3), J4.3 (Pin_3), J5.2 (Pin_2), J6.2 (Pin_2); no longer C1.2, U1.4 (V-)
- net at C12.1, C8.1, R6.1: now also U1.7; no longer U1.1
- net at C9.1, R11.2: now also U1.5 (+); no longer U1.2 (-)
- net at C8.2, R10.2: now also U1.6 (-); no longer U1.3 (+)
- net at C4.1, R11.1, R7.1: now also R3.1; no longer R2.1
- net at C6.1, R10.1, R6.2: now also R2.1; no longer R3.1
- net at C5.1, R13.1, R9.1: now also R5.1; no longer R4.1
- net at C7.1, R12.1, R8.2: now also R4.1; no longer R5.1
- net at C10.1, C13.1, R8.1: now also U1.1; no longer U1.7
- net at C10.2, R12.2: now also U1.2 (-); no longer U1.5 (+)
- net at C11.1, R13.2: now also U1.3 (+); no longer U1.6 (-)
- net at R1.1, U2.11 (~AUTO_MUTE), U2.12 (DIF2)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: now also J1.1 (G1), J2.1 (G1)
- net at U2.19 (DIF1): now also J2.2 (G2)
- net at U2.20 (DIF0): now also J1.2 (G2)
- net +12V renamed +15V
- net +15V: now also J4.1 (Pin_1)
- net L+: no longer names the net of FL1.3
- net L+: now also J5.1 (Pin_1)
- net L-: no longer names the net of FL2.3
- net L-: now also J5.3 (Pin_3)
- net R+: no longer names the net of FL3.3
- net R+: now also J6.1 (Pin_1)
- net R-: no longer names the net of FL4.3
- net R-: now also J6.3 (Pin_3)
Other:
- moved on the sheet: C1, C10, C11, C12, C13, C14, C15, C16, C17, C18, C19, C20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

Commit message: pre-trace
Parts:
- D1, D2, D3, D4: footprint Diodes_THT:D_A-405_P10.16mm_Horizontal -> Diodes_THT:D_DO-35_SOD27_P2.54mm_Vertical_AnodeUp
- J4: footprint (none) -> Pin_Headers:Pin_Header_Straight_1x04_Pitch2.54mm
- J5, J6: footprint (none) -> Connectors_Terminal_Blocks:TerminalBlock_Altech_AK300-3_P5.00mm
- R1, R10, R11, R12, R13, R2, R3, R4, R5, R6, R7, R8, R9: footprint Resistors_THT:R_Axial_DIN0207_L6.3mm_D2.5mm_P10.16mm_Horizontal -> Resistors_THT:R_Axial_DIN0204_L3.6mm_D1.6mm_P2.54mm_Vertical
Changed lines of the file:
@@
 F 0 "R6" V 5580 1600 50  0000 C CNN
 F 1 "13.7k" V 5500 1600 50  0000 C CNN
-F 2 "Resistors_THT:R_Axial_DIN0207_L6.3mm_D2.5mm_P10.16mm_Horizontal" V 5430 1600 50  0001 C CNN
+F 2 "Resistors_THT:R_Axial_DIN0204_L3.6mm_D1.6mm_P2.54mm_Vertical" V 5430 1600 50  0001 C CNN
 F 3 "" H 5500 1600 50  0001 C CNN
 	1    5500 1600
@@
 F 0 "R11" V 5980 2000 50  0000 C CNN
 F 1 "3,32k" V 5900 2000 50  0000 C CNN
-F 2 "Resistors_THT:R_Axial_DIN0207_L6.3mm_D2.5mm_P10.16mm_Horizontal" V 5830 2000 50  0001 C CNN
+F 2 "Resistors_THT:R_Axial_DIN0204_L3.6mm_D1.6mm_P2.54mm_Vertical" V 5830 2000 50  0001 C CNN
 F 3 "" H 5900 2000 50  0001 C CNN
 	1    5900 2000
@@
 F 0 "R10" V 5980 1800 50  0000 C CNN
 F 1 "3.32k" V 5900 1800 50  0000 C CNN
-F 2 "Resistors_THT:R_Axial_DIN0207_L6.3mm_D2.5mm_P10.16mm_Horizontal" V 5830 1800 50  0001 C CNN
+F 2 "Resistors_THT:R_Axial_DIN0204_L3.6mm_D1.6mm_P2.54mm_Vertical" V 5830 1800 50  0001 C CNN
 F 3 "" H 5900 1800 50  0001 C CNN
 	1    5900 1800
@@
 F 0 "R7" V 5580 2200 50  0000 C CNN
 F 1 "13.7k" V 5500 2200 50  0000 C CNN
-F 2 "Resistors_THT:R_Axial_DIN0207_L6.3mm_D2.5mm_P10.16mm_Horizontal" V 5430 2200 50  0001 C CNN
+F 2 "Resistors_THT:R_Axial_DIN0204_L3.6mm_D1.6mm_P2.54mm_Vertical" V 5430 2200 50  0001 C CNN
 F 3 "" H 5500 2200 50  0001 C CNN
 	1    5500 2200
@@
 F 0 "R8" V 5580 3550 50  0000 C CNN
 F 1 "13.7k" V 5500 3550 50  0000 C CNN
-F 2 "Resistors_THT:R_Axial_DIN0207_L6.3mm_D2.5mm_P10.16mm_Horizontal" V 5430 3550 50  0001 C CNN
+F 2 "Resistors_THT:R_Axial_DIN0204_L3.6mm_D1.6mm_P2.54mm_Vertical" V 5430 3550 50  0001 C CNN
 F 3 "" H 5500 3550 50  0001 C CNN
 	1    5500 3550
@@
 F 0 "R13" V 5980 3950 50  0000 C CNN
 F 1 "3.32k" V 5900 3950 50  0000 C CNN
-F 2 "Resistors_THT:R_Axial_DIN0207_L6.3mm_D2.5mm_P10.16mm_Horizontal" V 5830 3950 50  0001 C CNN
+F 2 "Resistors_THT:R_Axial_DIN0204_L3.6mm_D1.6mm_P2.54mm_Vertical" V 5830 3950 50  0001 C CNN
 F 3 "" H 5900 3950 50  0001 C CNN
 	1    5900 3950
@@
 F 0 "R12" V 5980 3750 50  0000 C CNN
 F 1 "3.32k" V 5900 3750 50  0000 C CNN
-F 2 "Resistors_THT:R_Axial_DIN0207_L6.3mm_D2.5mm_P10.16mm_Horizontal" V 5830 3750 50  0001 C CNN
+F 2 "Resistors_THT:R_Axial_DIN0204_L3.6mm_D1.6mm_P2.54mm_Vertical" V 5830 3750 50  0001 C CNN
 F 3 "" H 5900 3750 50  0001 C CNN
 	1    5900 3750
@@
 F 0 "R9" V 5580 4150 50  0000 C CNN
 F 1 "13.7kR" V 5500 4150 50  0000 C CNN
-F 2 "Resistors_THT:R_Axial_DIN0207_L6.3mm_D2.5mm_P10.16mm_Horizontal" V 5430 4150 50  0001 C CNN
+F 2 "Resistors_THT:R_Axial_DIN0204_L3.6mm_D1.6mm_P2.54mm_Vertical" V 5430 4150 50  0001 C CNN
 F 3 "" H 5500 4150 50  0001 C CNN
 	1    5500 4150
@@
 F 0 "D1" H 9250 1550 50  0000 C CNN
 F 1 "D" H 9250 1350 50  0000 C CNN
-F 2 "Diodes_THT:D_A-405_P10.16mm_Horizontal" H 9250 1450 50  0001 C CNN
+F 2 "Diodes_THT:D_DO-35_SOD27_P2.54mm_Vertical_AnodeUp" H 9250 1450 50  0001 C CNN
 F 3 "" H 9250 1450 50  0001 C CNN
 	1    9250 1450
@@
 F 0 "D3" H 9550 1550 50  0000 C CNN
 F 1 "D" H 9550 1350 50  0000 C CNN
-F 2 "Diodes_THT:D_A-405_P10.16mm_Horizontal" H 9550 1450 50  0001 C CNN
+F 2 "Diodes_THT:D_DO-35_SOD27_P2.54mm_Vertical_AnodeUp" H 9550 1450 50  0001 C CNN
 F 3 "" H 9550 1450 50  0001 C CNN
 	1    9550 1450
@@
 F 0 "D2" H 9250 3500 50  0000 C CNN
 F 1 "D" H 9250 3300 50  0000 C CNN
-F 2 "Diodes_THT:D_A-405_P10.16mm_Horizontal" H 9250 3400 50  0001 C CNN
+F 2 "Diodes_THT:D_DO-35_SOD27_P2.54mm_Vertical_AnodeUp" H 9250 3400 50  0001 C CNN
 F 3 "" H 9250 3400 50  0001 C CNN
 	1    9250 3400
@@
 F 0 "D4" H 9550 3500 50  0000 C CNN
 F 1 "D" H 9550 3300 50  0000 C CNN
-F 2 "Diodes_THT:D_A-405_P10.16mm_Horizontal" H 9550 3400 50  0001 C CNN
+F 2 "Diodes_THT:D_DO-35_SOD27_P2.54mm_Vertical_AnodeUp" H 9550 3400 50  0001 C CNN
 F 3 "" H 9550 3400 50  0001 C CNN
 	1    9550 3400
@@
 F 0 "R3" V 4130 3250 50  0000 C CNN
 F 1 "13.7k" V 4050 3250 50  0000 C CNN
-F 2 "Resistors_THT:R_Axial_DIN0207_L6.3mm_D2.5mm_P10.16mm_Horizontal" V 3980 3250 50  0001 C CNN
+F 2 "Resistors_THT:R_Axial_DIN0204_L3.6mm_D1.6mm_P2.54mm_Vertical" V 3980 3250 50  0001 C CNN
 F 3 "" H 4050 3250 50  0001 C CNN
 	1    4050 3250
@@
 F 0 "R2" V 4130 3050 50  0000 C CNN
 F 1 "13.7k" V 4050 3050 50  0000 C CNN
-F 2 "Resistors_THT:R_Axial_DIN0207_L6.3mm_D2.5mm_P10.16mm_Horizontal" V 3980 3050 50  0001 C CNN
+F 2 "Resistors_THT:R_Axial_DIN0204_L3.6mm_D1.6mm_P2.54mm_Vertical" V 3980 3050 50  0001 C CNN
 F 3 "" H 4050 3050 50  0001 C CNN
 	1    4050 3050
@@
 F 0 "R4" V 4130 3500 50  0000 C CNN
 F 1 "13.7k" V 4050 3500 50  0000 C CNN
-F 2 "Resistors_THT:R_Axial_DIN0207_L6.3mm_D2.5mm_P10.16mm_Horizontal" V 3980 3500 50  0001 C CNN
+F 2 "Resistors_THT:R_Axial_DIN0204_L3.6mm_D1.6mm_P2.54mm_Vertical" V 3980 3500 50  0001 C CNN
 F 3 "" H 4050 3500 50  0001 C CNN
 	1    4050 3500
@@
 F 0 "R5" V 4130 3700 50  0000 C CNN
 F 1 "13.7k" V 4050 3700 50  0000 C CNN
-F 2 "Resistors_THT:R_Axial_DIN0207_L6.3mm_D2.5mm_P10.16mm_Horizontal" V 3980 3700 50  0001 C CNN
+F 2 "Resistors_THT:R_Axial_DIN0204_L3.6mm_D1.6mm_P2.54mm_Vertical" V 3980 3700 50  0001 C CNN
 F 3 "" H 4050 3700 50  0001 C CNN
 	1    4050 3700
@@
 F 0 "R1" V 1980 3700 50  0000 C CNN
 F 1 "1k" V 1900 3700 50  0000 C CNN
-F 2 "Resistors_THT:R_Axial_DIN0207_L6.3mm_D2.5mm_P10.16mm_Horizontal" V 1830 3700 50  0001 C CNN
+F 2 "Resistors_THT:R_Axial_DIN0204_L3.6mm_D1.6mm_P2.54mm_Vertical" V 1830 3700 50  0001 C CNN
 F 3 "" H 1900 3700 50  0001 C CNN
 	1    1900 3700
@@
 F 0 "J4" H 8700 5600 50  0000 C CNN
 F 1 "Power In" H 8700 5100 50  0000 C CNN
-F 2 "" H 8700 5400 50  0001 C CNN
+F 2 "Pin_Headers:Pin_Header_Straight_1x04_Pitch2.54mm" H 8700 5400 50  0001 C CNN
 F 3 "" H 8700 5400 50  0001 C CNN
 	1    8700 5400
@@
 F 0 "J5" H 10500 2200 50  0000 C CNN
 F 1 "Left" H 10500 1800 50  0000 C CNN
-F 2 "" H 10500 2000 50  0001 C CNN
+F 2 "Connectors_Terminal_Blocks:TerminalBlock_Altech_AK300-3_P5.00mm" H 10500 2000 50  0001 C CNN
 F 3 "" H 10500 2000 50  0001 C CNN
 	1    10500 2000
@@
 F 0 "J6" H 10500 4150 50  0000 C CNN
 F 1 "Right" H 10500 3750 50  0000 C CNN
-F 2 "" H 10500 3950 50  0001 C CNN
+F 2 "Connectors_Terminal_Blocks:TerminalBlock_Altech_AK300-3_P5.00mm" H 10500 3950 50  0001 C CNN
 F 3 "" H 10500 3950 50  0001 C CNN
 	1    10500 3950

Commit message: base placement
Parts:
- J5, J6: footprint Connectors_Terminal_Blocks:TerminalBlock_Altech_AK300-3_P5.00mm -> Connectors_Molex:Molex_SPOX-5267_22-03-5035_03x2.54mm_Straight
Changed lines of the file:
@@
 $EndComp
-Wire Wire Line
-	2300 3700 2300 4800
 Wire Wire Line
 	2300 4100 2650 4100
@@
 F 0 "J5" H 10500 2200 50  0000 C CNN
 F 1 "Left" H 10500 1800 50  0000 C CNN
-F 2 "Connectors_Terminal_Blocks:TerminalBlock_Altech_AK300-3_P5.00mm" H 10500 2000 50  0001 C CNN
+F 2 "Connectors_Molex:Molex_SPOX-5267_22-03-5035_03x2.54mm_Straight" H 10500 2000 50  0001 C CNN
 F 3 "" H 10500 2000 50  0001 C CNN
 	1    10500 2000
@@
 F 0 "J6" H 10500 4150 50  0000 C CNN
 F 1 "Right" H 10500 3750 50  0000 C CNN
-F 2 "Connectors_Terminal_Blocks:TerminalBlock_Altech_AK300-3_P5.00mm" H 10500 3950 50  0001 C CNN
+F 2 "Connectors_Molex:Molex_SPOX-5267_22-03-5035_03x2.54mm_Straight" H 10500 3950 50  0001 C CNN
 F 3 "" H 10500 3950 50  0001 C CNN
 	1    10500 3950
@@
 Wire Wire Line
 	1350 4800 1350 4600
-Connection ~ 2300 4800
 Wire Wire Line
 	1850 4600 1850 4800
@@
 Wire Notes Line
 	1450 1800 1450 1100
+Wire Wire Line
+	2300 3700 2300 4800
+Connection ~ 2300 4800
 $EndSCHEMATC

Commit message: ready for prod
Parts:
- removed C14, C17: 1uF, Capacitors_THT:C_Rect_L7.2mm_W3.5mm_P5.00mm_FKS2_FKP2_MKS2_MKP2, symbol C
Changed lines of the file:
@@
 L GNDA #PWR05
 U 1 1 5AABCBAD
-P 7900 4450
-F 0 "#PWR05" H 7900 4200 50  0001 C CNN
-F 1 "GNDA" H 7900 4300 50  0000 C CNN
-F 2 "" H 7900 4450 50  0001 C CNN
-F 3 "" H 7900 4450 50  0001 C CNN
-	1    7900 4450
-	0    1    1    0
+P 7950 4450
+F 0 "#PWR05" H 7950 4200 50  0001 C CNN
+F 1 "GNDA" H 7950 4300 50  0000 C CNN
+F 2 "" H 7950 4450 50  0001 C CNN
+F 3 "" H 7950 4450 50  0001 C CNN
+	1    7950 4450
+	1    0    0    -1
 $EndComp
 $Comp
@@
 $EndComp
 $Comp
-L C C17
-U 1 1 5AABCBB9
-P 8150 4450
-F 0 "C17" H 8175 4550 50  0000 L CNN
-F 1 "1uF" H 8175 4350 50  0000 L CNN
-F 2 "Capacitors_THT:C_Rect_L7.2mm_W3.5mm_P5.00mm_FKS2_FKP2_MKS2_MKP2" H 8188 4300 50  0001 C CNN
-F 3 "" H 8150 4450 50  0001 C CNN
-	1    8150 4450
-	0    -1   -1   0
-$EndComp
-$Comp
 L -12V #PWR20
 U 1 1 5AABCBBF
-P 8550 4450
-F 0 "#PWR20" H 8550 4325 50  0001 C CNN
-F 1 "-15V" H 8550 4600 50  0000 C CNN
-F 2 "" H 8550 4450 50  0001 C CNN
-F 3 "" H 8550 4450 50  0001 C CNN
-	1    8550 4450
+P 8350 4450
+F 0 "#PWR20" H 8350 4325 50  0001 C CNN
+F 1 "-15V" H 8350 4600 50  0000 C CNN
+F 2 "" H 8350 4450 50  0001 C CNN
+F 3 "" H 8350 4450 50  0001 C CNN
+	1    8350 4450
 	-1   0    0    1
 $EndComp
@@
 $EndComp
 $Comp
-L GNDA #PWR06
-U 1 1 5AAC1046
-P 7900 1500
-F 0 "#PWR06" H 7900 1250 50  0001 C CNN
-F 1 "GNDA" H 7900 1350 50  0000 C CNN
-F 2 "" H 7900 1500 50  0001 C CNN
-F 3 "" H 7900 1500 50  0001 C CNN
-	1    7900 1500
-	0    1    1    0
-$EndComp
-$Comp
 L GNDA #PWR07
 U 1 1 5AAC104C
@@
 $EndComp
 $Comp
-L C C14
-U 1 1 5AAC1052
-P 8150 1500
-F 0 "C14" H 8175 1600 50  0000 L CNN
-F 1 "1uF" H 8175 1400 50  0000 L CNN
-F 2 "Capacitors_THT:C_Rect_L7.2mm_W3.5mm_P5.00mm_FKS2_FKP2_MKS2_MKP2" H 8188 1350 50  0001 C CNN
-F 3 "" H 8150 1500 50  0001 C CNN
-	1    8150 1500
-	0    -1   -1   0
-$EndComp
-$Comp
 L C C15
 U 1 1 5AAC1058
@@
 Connection ~ 8550 3600
 Wire Wire Line
-	8300 4450 8550 4450
-Wire Wire Line
-	7900 4450 8000 4450
-Wire Wire Line
 	7900 3450 8000 3450
 Wire Wire Line
@@
 Wire Wire Line
 	8350 4450 8350 4250
-Connection ~ 8350 4450
 Wire Wire Line
 	7150 1900 7500 1900
@@
 Wire Wire Line
 	7900 2500 8000 2500
-Wire Wire Line
-	8000 1500 7900 1500
 Connection ~ 7950 2500
 Wire Wire Line
@@
 	8550 2350 8550 2300
 Connection ~ 8550 2350
-Wire Wire Line
-	8300 1500 8550 1500
-Connection ~ 8350 1500
 Wire Wire Line
 	8350 1500 8350 1700
@@
 L +15V #PWR017
 U 1 1 5AB9ECD3
-P 8550 1500
-F 0 "#PWR017" H 8550 1350 50  0001 C CNN
-F 1 "+15V" H 8550 1640 50  0000 C CNN
-F 2 "" H 8550 1500 50  0001 C CNN
-F 3 "" H 8550 1500 50  0001 C CNN
-	1    8550 1500
+P 8350 1500
+F 0 "#PWR017" H 8350 1350 50  0001 C CNN
+F 1 "+15V" H 8350 1640 50  0000 C CNN
+F 2 "" H 8350 1500 50  0001 C CNN
+F 3 "" H 8350 1500 50  0001 C CNN
+	1    8350 1500
 	1    0    0    -1
 $EndComp
@@
 Wire Wire Line
 	7950 4050 7950 4450
-Connection ~ 7950 4450
 Wire Wire Line
 	9400 3150 9400 3200

Commit message: Rev B
Connections:
- net GNDA: no longer U2.1 (DEM0)
- net at C9.1, R11.2: now also U1.3 (+); no longer U1.5 (+)
- net at C8.2, R10.2: now also U1.2 (-); no longer U1.6 (-)
- net at C12.1, C8.1, R6.1: now also U1.1; no longer U1.7
- net L+: now reaches C4.1, R11.1, R3.1, R7.1
- net L-: now reaches C6.1, R10.1, R2.1, R6.2
- net R+: now reaches C5.1, R13.1, R5.1, R9.1
- net R-: now reaches C7.1, R12.1, R4.1, R8.2
- net at C10.1, C13.1, R8.1: now also U1.7; no longer U1.1
- net at C10.2, R12.2: now also U1.6 (-); no longer U1.2 (-)
- net at C11.1, R13.2: now also U1.5 (+); no longer U1.3 (+)
- net CTRL: now reaches J1.1 (G1), J2.1 (G1), R1.1, U2.11 (~AUTO_MUTE), U2.12 (DIF2), U2.15 (~MUTE_R), U2.16 (~MUTE_L), U2.2 (DEM1)
- net CTRL: now also U2.1 (DEM0)
- net -12V renamed -15V
Other:
- moved on the sheet: R1
Changed lines of the file:
@@
 L Opamp_Dual_Generic U1
 U 2 1 5AA919C7
-P 6850 1900
-F 0 "U1" H 6850 2100 50  0001 L CNN
-F 1 "OPA2604" H 6850 1700 50  0000 L CNN
-F 2 "Housings_DIP:DIP-8_W7.62mm_LongPads" H 6850 1900 50  0001 C CNN
-F 3 "" H 6850 1900 50  0001 C CNN
-	2    6850 1900
+P 6850 3850
+F 0 "U1" H 6850 4050 50  0001 L CNN
+F 1 "OPA2604" H 6850 3650 50  0000 L CNN
+F 2 "Housings_DIP:DIP-8_W7.62mm_LongPads" H 6850 3850 50  0001 C CNN
+F 3 "" H 6850 3850 50  0001 C CNN
+	2    6850 3850
 	1    0    0    1
 $EndComp
@@
 L Opamp_Dual_Generic U1
 U 1 1 5AAB91CA
-P 6850 3850
-F 0 "U1" H 6850 4050 50  0001 L CNN
-F 1 "OPA2604" H 6850 3650 50  0001 L CNN
-F 2 "Housings_DIP:DIP-8_W7.62mm_LongPads" H 6850 3850 50  0001 C CNN
-F 3 "" H 6850 3850 50  0001 C CNN
-	1    6850 3850
+P 6850 1900
+F 0 "U1" H 6850 2100 50  0001 L CNN
+F 1 "OPA2604" H 6850 1700 50  0001 L CNN
+F 2 "Housings_DIP:DIP-8_W7.62mm_LongPads" H 6850 1900 50  0001 C CNN
+F 3 "" H 6850 1900 50  0001 C CNN
+	1    6850 1900
 	1    0    0    1
 $EndComp
@@
 $EndComp
 $Comp
-L -12V #PWR20
+L -15V #PWR20
 U 1 1 5AABCBBF
 P 8350 4450
@@
 $EndComp
 $Comp
-L GNDA #PWR07
+L GNDA #PWR06
 U 1 1 5AAC104C
 P 7900 2500
-F 0 "#PWR07" H 7900 2250 50  0001 C CNN
+F 0 "#PWR06" H 7900 2250 50  0001 C CNN
 F 1 "GNDA" H 7900 2350 50  0000 C CNN
 F 2 "" H 7900 2500 50  0001 C CNN
@@
 $EndComp
 $Comp
-L -12V #PWR18
+L -15V #PWR18
 U 1 1 5AAC105E
 P 8550 2500
@@
 $EndComp
 $Comp
-L GNDA #PWR08
+L GNDA #PWR07
 U 1 1 5AAF4C8F
 P 8100 5550
-F 0 "#PWR08" H 8100 5300 50  0001 C CNN
+F 0 "#PWR07" H 8100 5300 50  0001 C CNN
 F 1 "GNDA" H 8100 5400 50  0000 C CNN
 F 2 "" H 8100 5550 50  0001 C CNN
@@
 $EndComp
 $Comp
-L +15V #PWR09
+L +15V #PWR08
 U 1 1 5AAF4E60
 P 8300 5200
-F 0 "#PWR09" H 8300 5050 50  0001 C CNN
+F 0 "#PWR08" H 8300 5050 50  0001 C CNN
 F 1 "+15V" H 8300 5340 50  0000 C CNN
 F 2 "" H 8300 5200 50  0001 C CNN
@@
 $EndComp
 $Comp
-L -12V #PWR16
+L -15V #PWR16
 U 1 1 5AAF4F22
 P 8300 5700
@@
 $EndComp
 $Comp
-L GNDA #PWR010
+L GNDA #PWR09
 U 1 1 5AAF6C77
 P 3400 4900
-F 0 "#PWR010" H 3400 4650 50  0001 C CNN
+F 0 "#PWR09" H 3400 4650 50  0001 C CNN
 F 1 "GNDA" H 3400 4750 50  0000 C CNN
 F 2 "" H 3400 4900 50  0001 C CNN
@@
 $EndComp
 $Comp
-L GNDA #PWR011
+L GNDA #PWR010
 U 1 1 5AAC510D
 P 9550 4000
-F 0 "#PWR011" H 9550 3750 50  0001 C CNN
+F 0 "#PWR010" H 9550 3750 50  0001 C CNN
 F 1 "GNDA" H 9550 3850 50  0000 C CNN
 F 2 "" H 9550 4000 50  0001 C CNN
@@
 $EndComp
 $Comp
-L GNDA #PWR012
+L GNDA #PWR011
 U 1 1 5AAC5235
 P 9550 2050
-F 0 "#PWR012" H 9550 1800 50  0001 C CNN
+F 0 "#PWR011" H 9550 1800 50  0001 C CNN
 F 1 "GNDA" H 9550 1900 50  0000 C CNN
 F 2 "" H 9550 2050 50  0001 C CNN
@@
 	3850 3700 3900 3700
 Wire Wire Line
-	4400 3250 4200 3250
+	4600 3250 4200 3250
 Connection ~ 7350 3850
 Wire Wire Line
@@
 	7800 1900 8150 1900
 Wire Wire Line
-	4400 3050 4200 3050
+	4500 3050 4200 3050
 Connection ~ 5150 3750
 Wire Wire Line
@@
 	3850 3900 4000 3900
 Wire Wire Line
-	4000 3900 4000 4800
+	4000 4800 4000 3900
 Wire Wire Line
 	3850 4000 4000 4000
@@
 Connection ~ 4000 4100
 Wire Wire Line
-	4000 4800 1350 4800
+	1350 4800 4000 4800
 Wire Wire Line
 	9050 1650 9050 1700
@@
 L R R1
 U 1 1 5AACAB31
-P 1900 3700
-F 0 "R1" V 1980 3700 50  0000 C CNN
-F 1 "1k" V 1900 3700 50  0000 C CNN
-F 2 "Resistors_THT:R_Axial_DIN0204_L3.6mm_D1.6mm_P2.54mm_Vertical" V 1830 3700 50  0001 C CNN
-F 3 "" H 1900 3700 50  0001 C CNN
-	1    1900 3700
+P 1850 3600
+F 0 "R1" V 1930 3600 50  0000 C CNN
+F 1 "1k" V 1850 3600 50  0000 C CNN
+F 2 "Resistors_THT:R_Axial_DIN0204_L3.6mm_D1.6mm_P2.54mm_Vertical" V 1780 3600 50  0001 C CNN
+F 3 "" H 1850 3600 50  0001 C CNN
+	1    1850 3600
 	0    1    1    0
 $EndComp
@@
 Connection ~ 2300 4100
 Wire Wire Line
-	2050 3700 2650 3700
-Wire Wire Line
-	2650 3600 2500 3600
-Wire Wire Line
-	2500 3600 2500 4650
+	2000 3600 2650 3600
 Wire Wire Line
 	1550 4650 3400 4650
@@
 SDATA
 $Comp
-L +5V #PWR013
+L +5V #PWR012
 U 1 1 5AACD882
-P 1600 3650
-F 0 "#PWR013" H 1600 3500 50  0001 C CNN
-F 1 "+5V" H 1600 3790 50  0000 C CNN
-F 2 "" H 1600 3650 50  0001 C CNN
-F 3 "" H 1600 3650 50  0001 C CNN
-	1    1600 3650
-	1    0    0    -1
-$EndComp
-Wire Wire Line
-	1600 3650 1600 3700
-Wire Wire Line
-	1600 3700 1750 3700
+P 1400 3600
+F 0 "#PWR012" H 1400 3450 50  0001 C CNN
+F 1 "+5V" H 1400 3740 50  0000 C CNN
+F 2 "" H 1400 3600 50  0001 C CNN
+F 3 "" H 1400 3600 50  0001 C CNN
+	1    1400 3600
+	1    0    0    -1
+$EndComp
+Wire Wire Line
+	1400 3600 1700 3600
 $Comp
 L EMI_Filter_LCL FL1
@@
 $EndComp
 $Comp
-L +5V #PWR014
+L +5V #PWR013
 U 1 1 5AACED81
 P 8100 5350
-F 0 "#PWR014" H 8100 5200 50  0001 C CNN
+F 0 "#PWR013" H 8100 5200 50  0001 C CNN
 F 1 "+5V" H 8100 5490 50  0000 C CNN
 F 2 "" H 8100 5350 50  0001 C CNN
@@
 $EndComp
 Wire Wire Line
-	4650 1800 4400 3050
-Wire Wire Line
-	4650 1800 5750 1800
-Wire Wire Line
-	4650 2000 5750 2000
-Wire Wire Line
-	4650 2000 4400 3250
-Wire Wire Line
-	4200 3500 4400 3500
-Wire Wire Line
-	4200 3700 4400 3700
-Wire Wire Line
-	4400 3700 4650 3950
-Wire Wire Line
-	4400 3500 4650 3750
+	4700 1800 4500 3050
+Wire Wire Line
+	4700 1800 5750 1800
+Wire Wire Line
+	4800 2000 5750 2000
+Wire Wire Line
+	4800 2000 4600 3250
+Wire Wire Line
+	4200 3500 4600 3500
+Wire Wire Line
+	4200 3700 4500 3700
+Wire Wire Line
+	4500 3700 4700 3950
+Wire Wire Line
+	4600 3500 4800 3750
 Wire Wire Line
 	1950 1300 1950 1050
@@
 Wire Wire Line
 	2050 4600 2050 4650
-Connection ~ 2500 4650
 Wire Wire Line
 	1550 4600 1550 4650
@@
 Connection ~ 2300 3700
 $Comp
-L +15V #PWR015
+L +15V #PWR014
 U 1 1 5AB9D852
 P 1650 1000
-F 0 "#PWR015" H 1650 850 50  0001 C CNN
+F 0 "#PWR014" H 1650 850 50  0001 C CNN
 F 1 "+15V" H 1650 1140 50  0000 C CNN
 F 2 "" H 1650 1000 50  0001 C CNN
@@
 $EndComp
 $Comp
-L -12V #PWR3
+L -15V #PWR3
 U 1 1 5AB9E2AD
 P 1650 1900
@@
 $EndComp
 $Comp
-L +15V #PWR016
+L +15V #PWR015
 U 1 1 5AB9EA60
 P 8550 3450
-F 0 "#PWR016" H 8550 3300 50  0001 C CNN
+F 0 "#PWR015" H 8550 3300 50  0001 C CNN
 F 1 "+15V" H 8550 3590 50  0000 C CNN
 F 2 "" H 8550 3450 50  0001 C CNN
@@
 $EndComp
 $Comp
-L +15V #PWR017
+L +15V #PWR016
 U 1 1 5AB9ECD3
 P 8350 1500
-F 0 "#PWR017" H 8350 1350 50  0001 C CNN
+F 0 "#PWR016" H 8350 1350 50  0001 C CNN
 F 1 "+15V" H 8350 1640 50  0000 C CNN
 F 2 "" H 8350 1500 50  0001 C CNN
@@
 $EndComp
 $Comp
-L +15V #PWR018
+L +15V #PWR017
 U 1 1 5AB9ED86
 P 9400 1200
-F 0 "#PWR018" H 9400 1050 50  0001 C CNN
+F 0 "#PWR017" H 9400 1050 50  0001 C CNN
 F 1 "+15V" H 9400 1340 50  0000 C CNN
 F 2 "" H 9400 1200 50  0001 C CNN
@@
 $EndComp
 $Comp
-L +15V #PWR019
+L +15V #PWR018
 U 1 1 5AB9EE39
 P 9400 3150
-F 0 "#PWR019" H 9400 3000 50  0001 C CNN
+F 0 "#PWR018" H 9400 3000 50  0001 C CNN
 F 1 "+15V" H 9400 3290 50  0000 C CNN
 F 2 "" H 9400 3150 50  0001 C CNN
@@
 	8300 5600 8500 5600
 Wire Wire Line
-	4650 3750 5750 3750
-Wire Wire Line
-	4650 3950 5750 3950
-$Comp
-L GNDA #PWR020
+	4800 3750 5750 3750
+Wire Wire Line
+	4700 3950 5750 3950
+$Comp
+L GNDA #PWR019
 U 1 1 5ABA37CC
 P 4050 2750
-F 0 "#PWR020" H 4050 2500 50  0001 C CNN
+F 0 "#PWR019" H 4050 2500 50  0001 C CNN
 F 1 "GNDA" H 4050 2600 50  0000 C CNN
 F 2 "" H 4050 2750 50  0001 C CNN
@@
 	1450 1800 1450 1100
 Wire Wire Line
-	2300 3700 2300 4800
+	2300 3600 2300 4800
 Connection ~ 2300 4800
+Connection ~ 2300 3600
+Wire Wire Line
+	2650 3700 2300 3700
+Text GLabel 4500 3050 0    60   Input ~ 0
+L-
+Text GLabel 4600 3250 0    60   Input ~ 0
+L+
+Text GLabel 4600 3500 0    60   Input ~ 0
+R-
+Text GLabel 4500 3700 0    60   Input ~ 0
+R+
+Text GLabel 2300 3800 0    60   Input ~ 0
+CTRL
 $EndSCHEMATC
